File: OPC/OPC.kicad_pcb (KiCad board)
At the start: 4 copper layers, 160 x 100 mm, 39 parts, among them J1 Conn_01x01, J2 Conn_01x01, J3 Conn_01x01, J4 Conn_01x01, J5 Conn_01x01, U1 LM5165X

Commit message: Development
Parts:
- removed J1, J4, J5: Conn_01x01, TestPoint:TestPoint_Plated_Hole_D2.0mm
- removed R1, R3: 0R/5%/100mW, Resistor_SMD:R_0603_1608Metric_Pad0.98x0.95mm_HandSolder
- J2, J3: value Conn_01x01 -> 1715721; footprint TestPoint:TestPoint_Plated_Hole_D2.0mm -> TerminalBlock_Phoenix:TerminalBlock_Phoenix_MKDS-1,5-2_1x02_P5.00mm_Horizontal
- moved C3 181.1 mm to (219.0, 116.0)
- moved R2 181.1 mm to (219.0, 121.0)
- moved C2 38.0 mm to (225.0, 121.0)
- moved J3 21.0 mm to (227.2, 132.0), turned to 90 degrees
- moved H4 16.1 mm to (213.0, 59.0)
- moved H3 16.0 mm to (213.0, 148.0)
- moved L1 11.2 mm to (225.0, 111.0)
- moved U1 11.2 mm to (224.8, 116.4)
- moved C6 11.0 mm to (222.0, 105.0)
- moved C7 11.0 mm to (228.0, 105.0)
- moved C4 7.28 mm to (222.0, 100.0), turned to 180 degrees
- moved C5 2.24 mm to (228.0, 100.0)
- moved H1 2.00 mm to (77.0, 59.0)
- moved H2 2.00 mm to (77.0, 147.0)
- moved J2 1.27 mm to (227.2, 73.5), turned to 90 degrees
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Connections:
- J2 pad 1: Net-(J2-Pin_1) -> VD
- U1 pad 2: Net-(J2-Pin_1) -> VD
- U1 pad 7: Net-(J2-Pin_1) -> VD

Commit message: Development
Parts:
- removed C7: 22u/25V/X7R, Capacitor_SMD:C_1210_3225Metric_Pad1.33x2.70mm_HandSolder
- removed J3: 1715721, TerminalBlock_Phoenix:TerminalBlock_Phoenix_MKDS-1,5-2_1x02_P5.00mm_Horizontal
- removed L1: SRR5028-221Y, OPC:SRR5028
- removed R2: 133k/1%/100mW, Resistor_SMD:R_0603_1608Metric_Pad0.98x0.95mm_HandSolder
- added J1: 1715721, TerminalBlock_Phoenix:TerminalBlock_Phoenix_MKDS-1,5-2_1x02_P5.00mm_Horizontal, F.Cu at (226.2, 78.5)
- C3: value 47n/100V/X7R -> 22u/25V/X7R; footprint Capacitor_SMD:C_0603_1608Metric_Pad1.08x0.95mm_HandSolder -> Capacitor_SMD:C_1210_3225Metric_Pad1.33x2.70mm_HandSolder
- D1, D2, D3: value BAT43W-V -> SS14; footprint Diode_SMD:D_SOD-123 -> Diode_SMD:D_SMA; moved to B.Cu
- D4, D5, D6: value BAT43W-V -> SS14; footprint Diode_SMD:D_SOD-123 -> Diode_SMD:D_SMA
- U1: value LM5165X -> TSR1-2450E; footprint Package_SON:Texas_S-PVSON-N10_ThermalVias -> Converter_DCDC:Converter_DCDC_TRACO_TSR1-xxxxE_THT
- moved C1 189.4 mm to (226.0, 84.5)
- moved D3 133.6 mm to (181.0, 65.0), turned to -90 degrees
- moved D5 98.1 mm to (135.0, 65.0), turned to -90 degrees
- moved D2 87.6 mm to (135.0, 65.0), turned to -90 degrees
- moved J2 59.0 mm to (226.2, 132.5)
- moved D1 53.6 mm to (89.0, 65.0), turned to -90 degrees
- moved C2 33.0 mm to (226.0, 88.0)
- moved D6 23.1 mm to (181.0, 65.0), turned to -90 degrees
- moved U1 21.4 mm to (224.5, 95.0)
- moved C5 13.6 mm to (226.0, 113.5)
- moved C6 12.6 mm to (226.0, 117.0), turned to 0 degrees
- moved C3 11.8 mm to (226.1, 106.5)
- moved C4 10.8 mm to (226.0, 110.0), turned to 0 degrees
- moved D4 2.00 mm to (89.0, 65.0), turned to -90 degrees
Connections:
- C3 pad 1: Net-(U1-SS) -> Net-(J2-Pin_1)
- C4 pad 1: Net-(J3-Pin_1) -> Net-(J2-Pin_1)
- C5 pad 1: Net-(J3-Pin_1) -> Net-(J2-Pin_1)
- C6 pad 1: Net-(J3-Pin_1) -> Net-(J2-Pin_1)
- J2 pad 1: VD -> Net-(J2-Pin_1)
- U1 pad 1: Net-(U1-SW) -> VD
- U1 pad 2: VD -> GND
- U1 pad 3: GND -> Net-(J2-Pin_1)
Routing:
- net Net-(SC7--): track 0.00 -> 70.5 mm
- net Net-(SC5--): track 0.00 -> 70.5 mm
- net Net-(SC3--): track 0.00 -> 70.5 mm
- net Net-(SC11--): track 0.00 -> 70.5 mm
- net Net-(SC10-+): track 0.00 -> 70.5 mm
- net Net-(SC1--): track 0.00 -> 70.5 mm
- net Net-(J2-Pin_1): track 0.00 -> 37.6 mm
- net VD: track 0.00 -> 17.2 mm
- net GND: vias 0 -> 1
- added copper zone on B.Cu, net GND
- added copper zone on F.Cu, net GND
Other:
- copper layers 4 -> 2

Commit message: Development
Routing:
- net VD: track 17.2 -> 71.4 mm, vias 0 -> 10
- added copper zone on B.Cu, net Net-(D1-A)
- added copper zone on B.Cu, net Net-(D2-A)
- added copper zone on B.Cu, net Net-(D3-A)
- added copper zone on F.Cu, net Net-(D4-A)
- added copper zone on F.Cu, net Net-(D5-A)
- added copper zone on F.Cu, net Net-(D6-A)
- added copper zone on B.Cu, net VD
- added copper zone on F.Cu, net VD

Commit message: Development
Routing:
- net Net-(J2-Pin_1): track 37.6 -> 35.9 mm
- net GND: vias 1 -> 16
Other:
- outline, holes or cut-outs redrawn
- board text added: "OPC"

Commit message: Development
Parts:
- moved C2 7.28 mm to (228.0, 95.0)
- moved C1 6.09 mm to (228.0, 90.2)
- moved U1 5.77 mm to (226.2, 100.5)
- moved C4 5.30 mm to (227.8, 115.0)
- moved C5 5.30 mm to (227.8, 118.5)
- moved C6 5.30 mm to (227.8, 122.0)
- moved C3 5.28 mm to (227.8, 111.5)
- moved J1 3.35 mm to (227.0, 81.8)
- moved H2 1.00 mm to (77.0, 148.0)
- moved J2 0.83 mm to (227.0, 132.5)
Routing:
- net Net-(J2-Pin_1): track 35.9 -> 63.6 mm
- net VD: track 71.4 -> 76.9 mm
- net GND: vias 16 -> 21
Other:
- outline, holes or cut-outs redrawn

Commit message: Design done
Other:
- board text added: "5V"
Changed lines of the file:
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@@
+	)
+	(gr_line
+		(start 218 75.25)
+		(end 218 78.25)
+		(stroke
+			(width 0.5)
+			(type default)
+		)
+		(layer "F.SilkS")
+	)
+	(gr_line
+		(start 218 80.25)
+		(end 218 83.25)
+		(stroke
+			(width 0.5)
+			(type default)
+		)
+		(layer "F.SilkS")
+	)
+	(gr_line
+		(start 218 126)
+		(end 218 129)
+		(stroke
+			(width 0.5)
+			(type default)
+		)
+		(layer "F.SilkS")
+	)
+	(gr_line
+		(start 218 131)
+		(end 218 134)
+		(stroke
+			(width 0.5)
+			(type default)
+		)
+		(layer "F.SilkS")
+	)
+	(gr_line
+		(start 219.5 81.75)
+		(end 216.5 81.75)
+		(stroke
+			(width 0.5)
+			(type default)
+		)
+		(layer "F.SilkS")
+	)
+	(gr_line
+		(start 219.5 132.5)
+		(end 216.5 132.5)
+		(stroke
+			(width 0.5)
+			(type default)
+		)
+		(layer "F.SilkS")
 	)
 	(gr_line
@@
 		(layer "Edge.Cuts")
 	)
-	(gr_rect
-		(start 78 70.5)
-		(end 215 135.5)
+	(gr_circle
+		(center 77 59)
+		(end 74 59)
 		(stroke
 			(width 0.1)
@@
 		(layer "User.1")
 	)
+	(gr_circle
+		(center 77 148)
+		(end 74 148)
+		(stroke
+			(width 0.1)
+			(type default)
+		)
+		(fill no)
+		(layer "User.1")
+	)
+	(gr_circle
+		(center 213 59)
+		(end 210 59)
+		(stroke
+			(width 0.1)
+			(type default)
+		)
+		(fill no)
+		(layer "User.1")
+	)
+	(gr_circle
+		(center 213 148)
+		(end 210 148)
+		(stroke
+			(width 0.1)
+			(type default)
+		)
+		(fill no)
+		(layer "User.1")
+	)
+	(gr_text "5V"
+		(at 222.75 142.25 0)
+		(layer "F.SilkS")
+		(effects
+			(font
+				(size 4 4)
+				(thickness 0.8)
+				(bold yes)
+			)
+			(justify left bottom)
+		)
+	)
 	(gr_text "OPC"
