File: OPC/OPC.kicad_sch (KiCad schematic)
At the start: 39 parts, among them J1 Conn_01x01, J2 Conn_01x01, J3 Conn_01x01, J4 Conn_01x01, J5 Conn_01x01, U1 LM5165X

Commit message: Development
Parts:
- removed J1, J2, J3, J4, J5: Conn_01x01, TestPoint:TestPoint_Plated_Hole_D2.0mm, symbol Connector_Generic:Conn_01x01
- removed R1, R3: 0R/5%/100mW, Resistor_SMD:R_0603_1608Metric_Pad0.98x0.95mm_HandSolder, symbol Device:R
- added J2, J3: 1715721, TerminalBlock_Phoenix:TerminalBlock_Phoenix_MKDS-1,5-2_1x02_P5.00mm_Horizontal, symbol Connector_Generic:Conn_01x02
Connections:
- net GND: now also J2.2 (Pin_2), J3.2 (Pin_2)
- net VD: now also U1.2 (VIN), U1.7 (EN), J2.1 (Pin_1)
- net at C4.1, C5.1, C6.1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: now also J3.1 (Pin_1)
Other:
- note removed: "Current measurement"
- note removed: "Voltage measurement"
- moved on the sheet: C1, C2, C3, C4, C5, C6, C7, D1, D2, D3, D4, D5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

Commit message: Development
Parts:
- removed C3: 47n/100V/X7R, Capacitor_SMD:C_0603_1608Metric_Pad1.08x0.95mm_HandSolder, symbol Device:C
- removed D1, D2, D3, D4, D5, D6: BAT43W-V, Diode_SMD:D_SOD-123, symbol Diode:BAT43W-V
- removed L1: SRR5028-221Y, OPC:SRR5028, symbol Device:L
- removed R2: 133k/1%/100mW, Resistor_SMD:R_0603_1608Metric_Pad0.98x0.95mm_HandSolder, symbol Device:R
- removed U1: LM5165X, Package_SON:Texas_S-PVSON-N10_ThermalVias, symbol Regulator_Switching:LM5165X
- added D1, D2, D3, D4, D5, D6: SS14, Diode_SMD:D_SMA, symbol Diode:SS14
- added U1: TSR1-2450E, Converter_DCDC:Converter_DCDC_TRACO_TSR1-xxxxE_THT, symbol Converter_DCDC:TSR1-2450E
- renumbered C4 to C3, C5 to C4, C6 to C5, C7 to C6, J2 to J1, J3 to J2
Connections:
- net GND: now also U1.2 (GND)
- net VD: now also D1.1 (K), D2.1 (K), D3.1 (K), D4.1 (K), D5.1 (K), D6.1 (K), U1.1 (Vin)
- net at C3.1, C4.1, C5.1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: now also U1.3 (Vout)
- net at SC7.1 (+): now also D4.2 (A)
- net at SC9.1 (+): now also D5.2 (A)
- net at SC11.1 (+): now also D6.2 (A)
- net at SC3.1 (+): now also D2.2 (A)
- net at SC5.1 (+): now also D3.2 (A)
- net at SC1.1 (+): now also D1.2 (A)
- no-connect marks 2 -> 0
Other:
- note added: "MAX: 9V6/200mA"
- note removed: "MAX: 9V6/100mA"
- moved on the sheet: C3, C4, C5, C6, J2

Commit message: Development
Changed lines of the file:
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@@
+	)
+	(junction
+		(at 203.2 119.38)
+		(diameter 0)
+		(color 0 0 0 0)
 	)
 	(junction
@@
 	(wire
 		(pts
+			(xy 203.2 119.38) (xy 217.17 119.38)
+		)
+		(stroke
+			(width 0)
+			(type default)
+		)
+	)
+	(wire
+		(pts
 			(xy 237.49 119.38) (xy 241.3 119.38)
 		)
@@
 	(wire
 		(pts
+			(xy 227.33 149.86) (xy 227.33 151.13)
+		)
+		(stroke
+			(width 0)
+			(type default)
+		)
+	)
+	(wire
+		(pts
 			(xy 55.88 148.59) (xy 55.88 149.86)
 		)
@@
 	(wire
 		(pts
-			(xy 180.34 119.38) (xy 217.17 119.38)
+			(xy 180.34 119.38) (xy 203.2 119.38)
+		)
+		(stroke
+			(width 0)
+			(type default)
+		)
+	)
+	(wire
+		(pts
+			(xy 203.2 118.11) (xy 203.2 119.38)
 		)
 		(stroke
@@
 			(width 0)
 			(type default)
+		)
+	)
+	(symbol
+		(lib_id "power:PWR_FLAG")
+		(at 203.2 118.11 0)
+		(unit 1)
+		(body_style 1)
+		(exclude_from_sim no)
+		(in_bom yes)
+		(on_board yes)
+		(in_pos_files yes)
+		(dnp no)
+		(fields_autoplaced yes)
+		(property "Reference" "#FLG02"
+			(at 203.2 116.205 0)
+			(hide yes)
+			(show_name no)
+			(do_not_autoplace no)
+			(effects
+				(font
+					(size 1.27 1.27)
+				)
+			)
+		)
+		(property "Value" "PWR_FLAG"
+			(at 203.2 113.03 0)
+			(show_name no)
+			(do_not_autoplace no)
+			(effects
+				(font
+					(size 1.27 1.27)
+				)
+			)
+		)
+		(property "Footprint" ""
+			(at 203.2 118.11 0)
+			(hide yes)
+			(show_name no)
+			(do_not_autoplace no)
+			(effects
+				(font
+					(size 1.27 1.27)
+				)
+			)
+		)
+		(property "Datasheet" ""
+			(at 203.2 118.11 0)
+			(hide yes)
+			(show_name no)
+			(do_not_autoplace no)
+			(effects
+				(font
+					(size 1.27 1.27)
+				)
+			)
+		)
+		(property "Description" "Special symbol for telling ERC where power comes from"
+			(at 203.2 118.11 0)
+			(hide yes)
+			(show_name no)
+			(do_not_autoplace no)
+			(effects
+				(font
+					(size 1.27 1.27)
+				)
+			)
+		)
+		(pin "1"
+		)
+		(instances
+			(project "OPC"
+				(path "/5c55bdfc-b12e-4294-8d2f-813ebb68046e"
+					(reference "#FLG02")
+					(unit 1)
+				)
+			)
 		)
 	)
@@
 					(unit 1)
 				)
+			)
+		)
+	)
+	(symbol
+		(lib_id "power:PWR_FLAG")
+		(at 227.33 151.13 180)
+		(unit 1)
+		(body_style 1)
+		(exclude_from_sim no)
+		(in_bom yes)
+		(on_board yes)
+		(in_pos_files yes)
+		(dnp no)
+		(fields_autoplaced yes)
+		(property "Reference" "#FLG01"
+			(at 227.33 153.035 0)
+			(hide yes)
+			(show_name no)
+			(do_not_autoplace no)
+			(effects
+				(font
+					(size 1.27 1.27)
+				)
+			)
+		)
+		(property "Value" "PWR_FLAG"
+			(at 227.33 156.21 0)
+			(show_name no)
+			(do_not_autoplace no)
+			(effects
+				(font
+					(size 1.27 1.27)
+				)
+			)
+		)
+		(property "Footprint" ""
+			(at 227.33 151.13 0)
+			(hide yes)
+			(show_name no)
+			(do_not_autoplace no)
+			(effects
+				(font
+					(size 1.27 1.27)
+				)
+			)
+		)
+		(property "Datasheet" ""
+			(at 227.33 151.13 0)
+			(hide yes)
+			(show_name no)
+			(do_not_autoplace no)
+			(effects
+				(font
+					(size 1.27 1.27)
+				)
+			)
+		)
+		(property "Description" "Special symbol for telling ERC where power comes from"
+			(at 227.33 151.13 0)
+			(hide yes)
+			(show_name no)
+			(do_not_autoplace no)
+			(effects
+				(font
+					(size 1.27 1.27)
+				)
+			)
+		)
+		(pin "1"
+		)
+		(instances
+			(project "OPC"
+				(path "/5c55bdfc-b12e-4294-8d2f-813ebb68046e"
+					(reference "#FLG01")
+					(unit 1)
+				)

Commit message: Design done
Other:
- moved on the sheet: C1, C2, C3, C4, C5, C6, D1, D2, D3, D4, D5, D6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
