File: LED/LED.kicad_pcb (KiCad board)
At the start: 2 copper layers, 160 x 100 mm, 38 parts, among them J1 1715721, Q1 CSD18501Q5A, U1 OPA192IDR, U2 LM5165X

Commit message: Development
Parts:
- removed C4: 47n/100V/X7R, Capacitor_SMD:C_0603_1608Metric_Pad1.08x0.95mm_HandSolder
- removed L1: SRR5028-221Y, OPC:SRR5028
- removed R13: 133k/1%/100mW, Resistor_SMD:R_0603_1608Metric_Pad0.98x0.95mm_HandSolder
- U2: value LM5165X -> TSR1-2450E; footprint Package_SON:Texas_S-PVSON-N10_ThermalVias -> Converter_DCDC:Converter_DCDC_TRACO_TSR1-xxxxE_THT
Connections:
- C5 pad 1: Net-(U2-VOUT) -> Net-(U2-Vout)
- C6 pad 1: Net-(U2-VOUT) -> Net-(U2-Vout)
- R12 pad 1: Net-(U2-VOUT) -> Net-(U2-Vout)
- U2 pad 1: Net-(U2-SW) -> +24V
- U2 pad 2: +24V -> GND
- U2 pad 3: GND -> Net-(U2-Vout)

Commit message: Development
Parts:
- D1, D2, D3, D4, D5, D6, D7, D8: moved to B.Cu
- moved H3 134.1 mm to (213.0, 59.0)
- moved H4 129.6 mm to (213.0, 148.0)
- moved R10 114.3 mm to (212.2, 112.2), turned to -90 degrees
- moved C6 112.1 mm to (206.5, 98.0), turned to -90 degrees
- moved R11 111.9 mm to (210.2, 112.2), turned to -90 degrees
- moved R12 110.0 mm to (209.6, 97.2), turned to -90 degrees
- moved C5 108.2 mm to (199.8, 71.1), turned to 180 degrees
- moved U1 105.8 mm to (211.2, 103.8), turned to -90 degrees
- moved C3 101.2 mm to (193.5, 71.1)
- moved J1 100.0 mm to (184.8, 64.2), turned to 180 degrees
- moved U2 95.7 mm to (194.0, 65.0), turned to 90 degrees
- moved D5 90.3 mm to (96.0, 119.2), turned to 90 degrees
- moved Q1 78.6 mm to (210.8, 119.2), turned to 180 degrees
- moved D4 72.9 mm to (96.0, 86.8), turned to -90 degrees
- moved R5 65.9 mm to (96.0, 119.2)
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Other:
- board size 160 x 100 mm -> 148 x 100 mm
- board text added: "LED"

Commit message: Design done
Parts:
- moved D1 40.0 mm to (158.0, 86.8)
- moved D8 40.0 mm to (158.0, 119.2)
- moved R1 40.0 mm to (158.0, 86.8)
- moved R8 40.0 mm to (158.0, 119.2)
- moved D2 29.0 mm to (135.0, 86.8)
- moved D7 29.0 mm to (135.0, 119.2)
- moved R2 29.0 mm to (135.0, 86.8)
- moved R7 29.0 mm to (135.0, 119.2)
- moved Q1 26.5 mm to (184.2, 119.5)
- moved D3 18.0 mm to (112.0, 86.8)
- moved D6 18.0 mm to (112.0, 119.2)
- moved R3 18.0 mm to (112.0, 86.8)
- moved R6 18.0 mm to (112.0, 119.2)
- moved C1 17.0 mm to (194.2, 109.8)
- moved C2 17.0 mm to (198.0, 103.5)
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Routing:
- net +24V: track 0.00 -> 50.7 mm, vias 0 -> 10
- net Net-(U2-Vout): track 0.00 -> 40.2 mm
- net Net-(U1--): track 0.00 -> 10.5 mm, vias 0 -> 2
- net Net-(Q1-S-Pad1): track 0.00 -> 8.92 mm
- net Net-(Q1-G): track 0.00 -> 8.62 mm
- net Net-(C1-Pad1): track 0.00 -> 5.26 mm
- net Net-(U1-+): track 0.00 -> 5.18 mm
- net Net-(R14-Pad2): track 0.00 -> 1.75 mm
- net Net-(D8-K): vias 0 -> 9
- net Net-(D7-K): vias 0 -> 9
- net Net-(D6-K): vias 0 -> 9
- net Net-(D5-K): vias 0 -> 9
- net Net-(D4-K): vias 0 -> 8
- net Net-(D3-K): vias 0 -> 9
- net Net-(D2-K): vias 0 -> 9
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- added copper zone on B.Cu, net +24V
- added copper zone on F.Cu, net +24V
- added copper zone on B.Cu, net GND
- added copper zone on F.Cu, net GND
- added copper zone on B.Cu, net Net-(D1-K)
- added copper zone on F.Cu, net Net-(D1-K)
- added copper zone on B.Cu, net Net-(D2-K)
- added copper zone on F.Cu, net Net-(D2-K)
- added copper zone on B.Cu, net Net-(D3-K)
- added copper zone on F.Cu, net Net-(D3-K)
- added copper zone on B.Cu, net Net-(D4-K)
- added copper zone on F.Cu, net Net-(D4-K)
- added copper zone on B.Cu, net Net-(D5-K)
- added copper zone on F.Cu, net Net-(D5-K)
- added copper zone on B.Cu, net Net-(D6-K)
- added copper zone on F.Cu, net Net-(D6-K)
- added copper zone on B.Cu, net Net-(D7-K)
- added copper zone on F.Cu, net Net-(D7-K)
- added copper zone on B.Cu, net Net-(D8-K)
- added copper zone on F.Cu, net Net-(D8-K)
- added copper zone on F.Cu, net Net-(Q1-S-Pad1)
Other:
- board text added: "24V"
