File: LED/LED.kicad_sch (KiCad schematic)
At the start: 23 parts, among them Q1 CSD18501Q5A, U1 OPA192IDR

Commit message: Development
Parts:
- added C3, C5, C6: 22u/25V/X7R, Capacitor_SMD:C_1210_3225Metric_Pad1.33x2.70mm_HandSolder, symbol Device:C
- added C4: 47n/100V/X7R, Capacitor_SMD:C_0603_1608Metric_Pad1.08x0.95mm_HandSolder, symbol Device:C
- added H1, H2, H3, H4: MountingHole, MountingHole:MountingHole_3.2mm_M3_DIN965, symbol Mechanical:MountingHole
- added J1: 1715721, TerminalBlock_Phoenix:TerminalBlock_Phoenix_MKDS-1,5-2_1x02_P5.00mm_Horizontal, symbol Connector_Generic:Conn_01x02
- added L1: SRR5028-221Y, OPC:SRR5028, symbol Device:L
- added R12: 100k/0.1%/100mW, Resistor_SMD:R_0603_1608Metric_Pad0.98x0.95mm_HandSolder, symbol Device:R
- added R13: 133k/1%/100mW, Resistor_SMD:R_0603_1608Metric_Pad0.98x0.95mm_HandSolder, symbol Device:R
- added R14: 11k/0.1%/100mW, Resistor_SMD:R_0603_1608Metric_Pad0.98x0.95mm_HandSolder, symbol Device:R
- added R15: 110/0.1%/100mW, Resistor_SMD:R_0603_1608Metric_Pad0.98x0.95mm_HandSolder, symbol Device:R
- added U2: LM5165X, Package_SON:Texas_S-PVSON-N10_ThermalVias, symbol Regulator_Switching:LM5165X
- C1, C2: footprint (none) -> Capacitor_SMD:C_0603_1608Metric_Pad1.08x0.95mm_HandSolder
- D1, D2, D3, D4, D5, D6, D7, D8: footprint (none) -> OPC:SFH4715AS
- R1, R2, R3, R4, R5, R6, R7, R8: footprint (none) -> Resistor_SMD:R_2512_6332Metric_Pad1.40x3.35mm_HandSolder
- R10, R11: footprint (none) -> Resistor_SMD:R_0603_1608Metric_Pad0.98x0.95mm_HandSolder
- R9: value 1/1%/2W -> RNCL2512FT1R00; footprint (none) -> Resistor_SMD:R_2512_6332Metric_Pad1.40x3.35mm_HandSolder
Connections:
- net +24V: now also C3.1, J1.1 (Pin_1), U2.2 (VIN), U2.7 (EN)
- net GND: now also C3.2, C4.2, C5.2, C6.2, J1.2 (Pin_2), R13.2, R15.2, U2.10 (GND), U2.11 (GND), U2.3 (ILIM)
- net at R7.2, R8.1: now also D7.1 (K), D8.2 (A)
- net at U1.3 (+): now also R12.2, R14.1
- new net: R13.1, U2.5 (RT)
- new net: C4.1, U2.4 (SS)
- new net: C5.1, C6.1, L1.2, R12.1, U2.8 (VOUT)
- new net: R14.2, R15.1
- new net: L1.1, U2.1 (SW)
- no-connect marks 0 -> 2
Other:
- note removed: "https://www.analog.com/media/en/technical-documentation/data-sheets/max77505.pdf"
- moved on the sheet: C1, C2, D1, D2, D3, D4, D5, D6, D7, D8, Q1, R1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

Commit message: Development
Parts:
- removed C4: 47n/100V/X7R, Capacitor_SMD:C_0603_1608Metric_Pad1.08x0.95mm_HandSolder, symbol Device:C
- removed L1: SRR5028-221Y, OPC:SRR5028, symbol Device:L
- removed R13: 133k/1%/100mW, Resistor_SMD:R_0603_1608Metric_Pad0.98x0.95mm_HandSolder, symbol Device:R
- removed U2: LM5165X, Package_SON:Texas_S-PVSON-N10_ThermalVias, symbol Regulator_Switching:LM5165X
- added U2: TSR1-2450E, Converter_DCDC:Converter_DCDC_TRACO_TSR1-xxxxE_THT, symbol Converter_DCDC:TSR1-2450E
Connections:
- net +24V: now also U2.1 (Vin)
- net GND: now also U2.2 (GND)
- net at C5.1, C6.1, R12.1: now also U2.3 (Vout)
- no-connect marks 2 -> 0
Other:
- moved on the sheet: C2, C3, J1

Commit message: Design done
Other:
- note added: "Current set to 500 mA"
- moved on the sheet: C5, C6, H1, H2, H3, H4, R12, R14, R15, U2

Commit message: Updated README file
Parts:
- R1, R2, R3, R4, R5, R6, R7, R8: now not fitted
Changed lines of the file:
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@@
 		(on_board yes)
 		(in_pos_files yes)
-		(dnp no)
+		(dnp yes)
 		(fields_autoplaced yes)
 		(property "Reference" "R1"
@@
 		(on_board yes)
 		(in_pos_files yes)
-		(dnp no)
+		(dnp yes)
 		(fields_autoplaced yes)
 		(property "Reference" "R7"
@@
 		(on_board yes)
 		(in_pos_files yes)
-		(dnp no)
+		(dnp yes)
 		(fields_autoplaced yes)
 		(property "Reference" "R4"
@@
 		(on_board yes)
 		(in_pos_files yes)
-		(dnp no)
+		(dnp yes)
 		(fields_autoplaced yes)
 		(property "Reference" "R3"
@@
 		(on_board yes)
 		(in_pos_files yes)
-		(dnp no)
+		(dnp yes)
 		(fields_autoplaced yes)
 		(property "Reference" "R8"
@@
 		(on_board yes)
 		(in_pos_files yes)
-		(dnp no)
+		(dnp yes)
 		(fields_autoplaced yes)
 		(property "Reference" "R2"
@@
 		(on_board yes)
 		(in_pos_files yes)
-		(dnp no)
+		(dnp yes)
 		(fields_autoplaced yes)
 		(property "Reference" "R6"
@@
 		(on_board yes)
 		(in_pos_files yes)
-		(dnp no)
+		(dnp yes)
 		(fields_autoplaced yes)
 		(property "Reference" "R5"
